File: 5mm08_2p_for_breadboard.kicad_pcb (KiCad board)
At the start: 2 copper layers, 9.8 x 9.4 mm, 2 parts, among them J1 Conn_01x02, J2 Conn_02x02_Counter_Clockwise

Commit message: Apply KiCad6
Other:
- net class Default removed
